Commit message: Update robot description

File: frobit_description/urdf/frobit.urdf (robot description, URDF)
Before this commit: robot frobit, 3 links, 2 joints
Links:
- added link camera_link
- added link imu_link; visual box size=0.036 0.033 0.009
- added link left_wheel; visual cylinder length=0.02 radius=0.109
- added link right_wheel; visual cylinder length=0.02 radius=0.109
- link base_laser_link: geometry visual box size=0.06 0.06 0.075
- link lower_chassis: geometry visual box size=0.43 0.32 0.015
Joints:
- removed joint joint_lower_chassis_to_base_laser_link
- removed joint joint_lower_chassis_to_base_link
- added joint joint_base_laser: type fixed, parent lower_chassis, child base_laser_link, origin xyz=0.18 0 0.05 rpy=0 0 0
- added joint joint_camera: type fixed, parent lower_chassis, child camera_link, origin xyz=0.21 0.022 0.13 rpy=0 1.15 0
- added joint joint_imu: type fixed, parent lower_chassis, child imu_link, origin xyz=0.125 0 0.017 rpy=0 0 0
- added joint joint_left_wheel: type continuous, parent lower_chassis, child left_wheel, origin xyz=-0.105 -0.17 0 rpy=0 0 0, axis 0 1 0
- added joint joint_lower_chassis: type fixed, parent base_link, child lower_chassis, origin xyz=0.105 0 0 rpy=0 0 0
- added joint joint_right_wheel: type continuous, parent lower_chassis, child right_wheel, origin xyz=-0.105 0.17 0 rpy=0 0 0, axis 0 1 0

Commit message: Rename base_laser_link to laser_link for consistency

File: frobit_description/urdf/frobit.urdf (robot description, URDF)
Before this commit: robot frobit, 7 links, 6 joints
Links:
- removed link base_laser_link
- added link laser_link; visual box size=0.06 0.06 0.075
Joints:
- joint joint_base_laser: child base_laser_link -> laser_link

Commit message: Add base_footprint link to Frobit description

File: frobit_description/urdf/frobit.urdf (robot description, URDF)
Before this commit: robot frobit, 7 links, 6 joints
Links:
- added link base_footprint
Joints:
- added joint joint_base_footprint: type fixed, parent base_link, child base_footprint, origin xyz=0 0 -0.11650 rpy=0 0 0

Commit message: Update topic names and launch files correspondingly

File: frobit_description/urdf/frobit.urdf (robot description, URDF)
Before this commit: robot frobit, 8 links, 7 joints
Links:
- added link marker_link
Joints:
- added joint joint_marker_link: type fixed, parent lower_chassis, child marker_link, origin xyz=0 0 0 rpy=0 0 0

Commit message: Added 90 deg to camera angle

File: frobit_description/urdf/frobit.urdf (robot description, URDF)
Before this commit: robot frobit, 9 links, 8 joints
Joints:
- joint joint_camera: origin xyz=0.21 0.022 0.13 rpy=0 1.15 0 -> xyz=0.21 0.022 0.13 rpy=0 2.7053 0

Commit message: Camera frame angle corrected

File: frobit_description/urdf/frobit.urdf (robot description, URDF)
Before this commit: robot frobit, 9 links, 8 joints
Joints:
- joint joint_camera: origin xyz=0.21 0.022 0.13 rpy=0 2.7053 0 -> xyz=0.21 0.022 0.13 rpy=0 2.863853 0

Commit message: Update frobit description marker link

File: frobit_description/urdf/frobit.urdf (robot description, URDF)
Before this commit: robot frobit, 9 links, 8 joints
Links:
- link marker_link: geometry visual box size=0.2 0.2 0.01
Joints:
- joint joint_marker_link: origin xyz=0 0 0 rpy=0 0 0 -> xyz=-0.205 0 0.7 rpy=0 0 0

Commit message: Camera frame orientation corrected

File: frobit_description/urdf/frobit.urdf (robot description, URDF)
Before this commit: robot frobit, 9 links, 8 joints
Joints:
- joint joint_camera: origin xyz=0.21 0.022 0.13 rpy=0 2.863853 0 -> xyz=0.21 0.022 0.13 rpy=2.863853 0 1.57079632679
